File: RX.sch (KiCad schematic (older format))
At the start: 75 parts, among them J1 Conn_02x05_Top_Bottom, J3 SMA, J4 SMA, J5 From ADC VCM2 out, J6 To ADC Ain +/-, J7 From ADC VCM1 out, J8 To ADC Ain +/-, T3 TC4-1T/ WBC4-1TL, T4 TC4-1T/ WBC4-1TL, U10 LTC6400-20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

Commit message: schematic png added
Other:
- note added: "Red Pitaya 16 Frontend, RX section\n"
Changed lines of the file:
@@
 Wire Wire Line
 	2350 5000 3050 5000
+Text Notes 1300 3100 0    50   ~ 0
+Attenuator & Power In
+Text Notes 900  1550 0    50   ~ 0
+RX1 In
+Text Notes 800  3900 0    50   ~ 0
+RX2 In\n
 Wire Bus Line
 	2650 4050 2650 4250
@@
 Wire Bus Line
 	1850 2700 2050 2700
-Text Notes 1300 3100 0    50   ~ 0
-Attenuator & Power In
-Text Notes 900  1550 0    50   ~ 0
-RX1 In
-Text Notes 800  3900 0    50   ~ 0
-RX2 In\n
+Text Notes 6940 6880 0    157  ~ 31
+Red Pitaya 16 Frontend, RX section\n
 $EndSCHEMATC
