File: TX.sch (KiCad schematic (older format))
At the start: 78 parts, among them T1 1:1 Z, T2 1:1 Z, U1 OPA2677, U2 OPA2677

Commit message: schematic png added
Connections:
- wire segments 231 -> 230
Other:
- note added: "Red Pitaya 16 Frontend, TX section"
Changed lines of the file:
@@
 Wire Wire Line
 	4400 2130 4650 2130
-Wire Wire Line
-	4650 2970 4650 3230
 Connection ~ 4650 2130
 Wire Wire Line
 	4650 2130 4650 2270
-Connection ~ 4650 3230
 Wire Wire Line
-	4650 3230 4650 3450
+	4650 2970 4650 3450
+Text Notes 6950 6810 0    157  ~ 31
+Red Pitaya 16 Frontend, TX section
 $EndSCHEMATC
